File: MD/MD.kicad_sch (KiCad schematic)
At the start: 62 parts, among them J1 Conn_02x07_Odd_Even, J2 Conn_01x05_Pin, J3 Conn_01x05_Pin, J4 Conn_01x06_Pin, Q1 2SA1037AK, Q2 μPA2753GR, Q3 μPA2753GR, SW1 SW_Push, SW2 SW_DIP_x04, SW3 SW_SPDT, U1 RT9080-33GJ5, U2 STM32C011F4Px, U3 MAX3485, U4 IR2302, U5 IR2302, X1 MEMS_Oscillator_SiT2001B

Commit message: MDの回路を変更
Parts:
- removed Q1: 2SA1037AK, Package_TO_SOT_SMD:SOT-23-3, symbol Transistor_BJT:2SA1015
- added C13, C14: ~, Capacitor_SMD:C_0603_1608Metric_Pad1.08x0.95mm_HandSolder, symbol Device:C
- added C15, C16, C17, C18, C19, C20: 0.1uF, Capacitor_SMD:C_0603_1608Metric_Pad1.08x0.95mm_HandSolder, symbol Device:C
- added C21, C22: 10uF, Capacitor_SMD:C_0603_1608Metric_Pad1.08x0.95mm_HandSolder, symbol Device:C
- added D12, D13, D15: OSR50603C1E, LED_SMD:LED_0603_1608Metric_Pad1.05x0.95mm_HandSolder, symbol Device:LED
- added D16, D17, D19, D20, D21, D22: CUS01, Diode_SMD:D_SOD-323_HandSoldering, symbol Device:D_Schottky
- added D18: OSBL1608C1A, LED_SMD:LED_0603_1608Metric_Pad1.05x0.95mm_HandSolder, symbol Device:LED
- added J3: Conn_01x05_Pin, Connector_JST:JST_XH_B5B-XH-A_1x05_P2.50mm_Vertical, symbol Connector:Conn_01x05_Pin
- added J6: Conn_01x06_Pin, Connector_JST:JST_PH_B6B-PH-K_1x06_P2.00mm_Vertical, symbol Connector:Conn_01x06_Pin
- added J7: Conn_02x07_Odd_Even, Tomoshibi_Library:BoxHeader_2x07_P1.27mm_Vertical, symbol Connector_Generic:Conn_02x07_Odd_Even
- added Q1, Q4: 2SA1162, Package_TO_SOT_SMD:SOT-23-3, symbol Device:Q_PNP_BEC
- added Q5, Q6: μPA2753GR, Package_SO:SOP-8_3.9x4.9mm_P1.27mm, symbol Device:Q_Dual_NMOS_S1G1S2G2D2D2D1D1
- added R23: 7.5k, Resistor_SMD:R_0603_1608Metric_Pad0.98x0.95mm_HandSolder, symbol Device:R
- added R24: 20k, Resistor_SMD:R_0603_1608Metric_Pad0.98x0.95mm_HandSolder, symbol Device:R
- added R25: 6.8k, Resistor_SMD:R_0603_1608Metric_Pad0.98x0.95mm_HandSolder, symbol Device:R
- added R26, R27, R28: 2.2k, Resistor_SMD:R_0603_1608Metric_Pad0.98x0.95mm_HandSolder, symbol Device:R
- added R29, R35, R40: 1k, Resistor_SMD:R_0603_1608Metric_Pad0.98x0.95mm_HandSolder, symbol Device:R
- added R30, R31, R32, R33, R34, R41, R42, R43, R44: 10k, Resistor_SMD:R_0603_1608Metric_Pad0.98x0.95mm_HandSolder, symbol Device:R
- added R36, R37, R38, R39: 100, Resistor_SMD:R_0603_1608Metric_Pad0.98x0.95mm_HandSolder, symbol Device:R
- added SW4: SW_DIP_x04, Button_Switch_SMD:SW_DIP_SPSTx04_Slide_Copal_CHS-04B_W7.62mm_P1.27mm, symbol Switch:SW_DIP_x04
- added SW5: SW_Push, Button_Switch_SMD:SW_SPST_PTS810, symbol Switch:SW_Push
- added SW6: SW_SPDT, MyLibrary:SW_Slide_3P_SPDT, symbol Switch:SW_SPDT
- added TP2: TestPoint, TestPoint:TestPoint_THTPad_D2.0mm_Drill1.0mm, symbol Connector:TestPoint
- added U10: STM32C011F4Px, Package_SO:TSSOP-20_4.4x6.5mm_P0.65mm, symbol Tomoshibi_Library:STM32C011F4Px
- added U6: MAX3485, Package_SO:SOP-8_3.76x4.96mm_P1.27mm, symbol Interface_UART:MAX3485
- added U8, U9: IR2302, Package_SO:SOP-8_3.76x4.96mm_P1.27mm, symbol Driver_FET:IR2302
- added X2: MEMS_Oscillator_SiT2001B, Package_TO_SOT_SMD:SOT-23-5_HandSoldering, symbol Tomoshibi_Library:MEMS_Oscillator_SiT2001B
- J4: renamed from J1; footprint Tomoshibi_Library:BoxHeader_2x07_P1.27mm_Horizontal -> Tomoshibi_Library:BoxHeader_2x07_P1.27mm_Vertical
- SW1: footprint Button_Switch_SMD:SW_Push_1P1T_NO_6x6mm_H9.5mm -> Button_Switch_SMD:SW_SPST_PTS810
- SW3: footprint Tomoshibi_Library:SW_Slide_3P_SPDT -> MyLibrary:SW_Slide_3P_SPDT
- renumbered J2 to J1, J3 to J2, J4 to J5
Connections:
- net Main_A is gone; now on net MAIN_MD_A: J1.4 (Pin_4), J2.4 (Pin_4)
- net Main_B is gone; now on net MAIN_MD_B: J1.5 (Pin_5), J2.5 (Pin_5)
- net +12V: now also C18.1, C19.1, D12.2 (A), D16.2 (A), D17.2 (A), D19.1 (K), D21.1 (K), J3.2 (Pin_2), Q5.7 (D), Q5.8 (D), Q6.7 (D), Q6.8 (D), U8.1 (VCC), U9.1 (VCC)
- net +3.3V: now also C15.1, C16.1, C20.1, D15.2 (A), J7.3 (Pin_3), Q1.2 (E), Q4.2 (E), R27.1, R35.1, SW4.1, SW4.2, SW4.3, SW4.4, SW6.2 (B), U10.4 (VDD), U6.8 (VCC), X2.4 (VDD)
- net +5V: now also D13.2 (A), J3.3 (Pin_3), J6.4 (Pin_4)
- net GND: now also C13.2, C14.2, C15.2, C16.2, C17.1, C18.2, C19.2, C20.2, D20.2 (A), D22.2 (A), J3.1 (Pin_1), J6.3 (Pin_3), J7.11 (Pin_11), J7.5 (Pin_5), J7.7 (Pin_7), Q5.3 (S), Q6.3 (S), R24.2, R25.2, R26.2, R28.2, R29.2, R30.2, R31.2, R32.2, R33.2, R34.2, R40.2, R42.1, R44.1, SW5.2, TP2.1, U10.5 (VSS), U6.5 (GND), U8.4 (COM), U9.4 (COM), X2.1 (GND); no longer U2.2 (PC14), X1.5 (OUT)
- net at R5.2: now also Q1.1 (B)
- net DIPSW0 renamed DIPSW00
- net DIPSW1 renamed DIPSW01
- net DIPSW2 renamed DIPSW02
- net DIPSW3 renamed DIPSW03
- net Encorder_A renamed Encorder0_A
- net Encorder_B renamed Encorder0_B
- net LED renamed LED0
- net MD_A renamed MAIN_MD_A
- net MAIN_MD_A: now also J3.4 (Pin_4), R27.2, U6.6 (A)
- net MD_B renamed MAIN_MD_B
- net MAIN_MD_B: now also J3.5 (Pin_5), R28.1, U6.7 (B)
- net MD_RX/MAIN_TX renamed MD0_RX/MAIN_TX
- net MD0_RX/MAIN_TX: now also Q1.3 (C)
- net MD_TX/MAIN_RX renamed MD0_TX/MAIN_RX
- net Motor_A renamed Motor0_A
- net Motor_B renamed Motor0_B
- net NRST renamed NRST0
- net PWM_A renamed PWM0_A
- net PWM_B renamed PWM0_B
- net SHDN renamed SHDN0
- net SWCLK renamed SWCLK0
- net SWDIO renamed SWDIO0
- net SlideSW renamed SlideSW0
- new net: R38.1, U9.7 (HO)
- new net: Q6.2 (G), R38.2, R43.2
- new net: C21.1, D16.1 (K), U8.8 (VB)
- new net: C22.1, D17.1 (K), U9.8 (VB)
- new net: Q6.4 (G), R39.2, R44.2
- new net: R37.1, U8.5 (LO)
- new net: R36.1, U8.7 (HO)
- new net: Q5.2 (G), R36.2, R41.2
- new net: R39.1, U9.5 (LO)
- new net: R35.2, X2.3 (OE)
- new net: Q4.1 (B), R23.2
- new net: D18.1 (K), R40.1
- new net: D12.1 (K), R25.1
- new net: Q5.4 (G), R37.2, R42.2
- new net: D13.1 (K), R26.1
- new net: D15.1 (K), R29.1
- new net DIPSW10: R30.1, SW4.8, U10.17 (PA10/PA12)
- new net DIPSW11: R31.1, SW4.7, U10.16 (PA9/PA11)
- new net DIPSW12: R32.1, SW4.6, U10.15 (PA8)
- new net DIPSW13: R33.1, SW4.5, U10.13 (PA6)
- new net Encorder1_A: J6.2 (Pin_2), U10.1 (PB7)
- new net Encorder1_B: J6.1 (Pin_1), U10.14 (PA7)
- new net LED1: D18.2 (A), U10.9 (PA2)
- new net MD1_RX/MAIN_TX: Q4.3 (C), R24.1, U10.8 (PA1), U6.1 (RO), U6.2 (~{RE}), U6.3 (DE)
- new net MD1_TX/MAIN_RX: R23.1, U10.20 (PB6), U6.4 (DI)
- new net Motor1_A: C21.2, D19.2 (A), D20.1 (K), J6.6 (Pin_6), Q5.1 (S), Q5.5 (D), Q5.6 (D), R41.1, U8.6 (VS)
- new net Motor1_B: C22.2, D21.2 (A), D22.1 (K), J6.5 (Pin_5), Q6.1 (S), Q6.5 (D), Q6.6 (D), R43.1, U9.6 (VS)
- new net NRST1: C17.2, J7.12 (Pin_12), SW5.1, U10.6 (PF2)
- new net OSC0_IN: C13.1, U2.2 (PC14), X1.5 (OUT)
- new net OSC1_IN: C14.1, U10.2 (PC14), X2.5 (OUT)
- new net PWM1_A: U10.7 (PA0), U8.2 (IN)
- new net PWM1_B: U10.10 (PA3), U9.2 (IN)
- new net SHDN1: U10.3 (PC15), U8.3 (~{SD}), U9.3 (~{SD})
- new net SWCLK1: J7.6 (Pin_6), U10.19 (PA14)
- new net SWDIO1: J7.4 (Pin_4), U10.18 (PA13)
- new net SlideSW1: R34.1, SW6.1 (A), U10.12 (PA5)
- no-connect marks 9 -> 18
Other:
- note added: "MD1"
- note added: "MD2"
- note added: "システム"
- note added: "共通部分"
- note removed: "C011"
- note removed: "MEMS発振器"
- note removed: "NRST"
- note removed: "パスコン"
- note removed: "電源LED・テストポイント"
- moved on the sheet: C1, C10, C11, C12, C2, C3, C4, C5, C6, C7, C8, C9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
